File: kicad/k1-aioc/k1-aioc.kicad_sch (KiCad schematic)
At the start: 56 parts, among them J1 Conn_01x07_Male, J2 12401832E402A, J3 SIP 200, J4 SIP 200, U1 MIC5330-SSYML, U2 STM32F373CBTx(OLD), Y1 8MHz/20pF

Commit message: Updating PCB files
Parts:
- U3: value (none) -> 4N25
